File: LED/LED.kicad_pcb (KiCad board)
At the start: 2 copper layers, 100 x 100 mm, 25 parts, among them J1 USB_C_Receptacle_USB2.0, J2 RJ45, J3 RJ45, J4 Screw_Terminal_01x03, U1 CH340C, U2 WeMos_D1_mini, U3 ESP32-WROOM-32D, U4 AMS1117-3.3

Commit message: 2 ethernet
Parts:
- added SW1: SW_Push, Button_Switch_THT:SW_PUSH_6mm, F.Cu at (115.3, 88.2)
- moved R7 29.0 mm to (102.9, 69.8)
- moved J4 10.9 mm to (102.9, 86.4), turned to -90 degrees
- moved D1 9.23 mm to (75.9, 74.9)
- moved R5 7.11 mm to (97.8, 66.2)
- moved C1 5.24 mm to (102.9, 66.4)
- moved C4 4.55 mm to (75.7, 81.8)
- moved R4 4.33 mm to (100.8, 109.1), turned to 180 degrees
- moved U1 4.10 mm to (88.9, 67.0)
- moved U4 3.90 mm to (83.8, 81.3)
- moved R8 3.82 mm to (102.4, 77.5), turned to 180 degrees
- moved C2 3.78 mm to (97.3, 63.0)
- moved U2 3.55 mm to (72.9, 90.2)
- moved D4 3.46 mm to (97.8, 77.5)
- moved C5 3.45 mm to (91.4, 81.3)
- moved R6 3.01 mm to (102.4, 73.9)
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Connections:
- U3 pad 16: unconnected-(U3-Pad16) -> /SW1
Routing:
- net /PIN2_GOOD: track 0.00 -> 0.95 mm

Commit message: 2/12
first draft
Parts:
- removed J2: RJ45, WS_LCSC_Connectors:RJ45_5501-88011111
- moved SW1 8.98 mm to (124.2, 89.5)
- moved J4 3.81 mm to (106.7, 86.4)
- moved R6 0.20 mm to (102.4, 73.7), turned to 180 degrees
Connections:
- U3 pad 10: /PIN1_GOOD -> unconnected-(U3-Pad10)
- U3 pad 27: /PIN8_GOOD -> unconnected-(U3-Pad27)
- U3 pad 28: /PIN7_GOOD -> unconnected-(U3-Pad28)
- U3 pad 30: /PIN6_GOOD -> unconnected-(U3-Pad30)
- U3 pad 31: /PIN5_GOOD -> unconnected-(U3-Pad31)
- U3 pad 33: /PIN4_GOOD -> unconnected-(U3-Pad33)
- U3 pad 36: /PIN3_GOOD -> unconnected-(U3-Pad36)
- U3 pad 37: /PIN2_GOOD -> unconnected-(U3-Pad37)
Routing:
- net +3.3V: track 0.00 -> 71.5 mm, vias 0 -> 2
- net +5V: track 0.00 -> 67.7 mm
- net /GPI0O: track 0.00 -> 48.4 mm, vias 0 -> 2
- net +24V: track 0.00 -> 30.2 mm
- net /RST: track 0.00 -> 22.3 mm
- net Net-(D1-Pad2): track 0.00 -> 20.6 mm, vias 0 -> 2
- net /D+: track 0.00 -> 19.4 mm
- net /D-: track 0.00 -> 17.8 mm
- net /SW1: track 0.00 -> 15.2 mm
- net GND: track 0.00 -> 9.27 mm, vias 0 -> 2
- net Net-(R8-Pad1): track 0.00 -> 8.68 mm
- net Net-(R6-Pad1): track 0.00 -> 7.63 mm
- net Net-(R3-Pad1): track 0.00 -> 6.85 mm
- net /WEMOS_GND: track 0.00 -> 5.52 mm
- net Net-(D2-Pad2): track 0.00 -> 5.38 mm
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- added copper zone on B.Cu, net GND
- added copper zone on F.Cu, net GND

Commit message: to gnd
Connections:
- D3 pad 1: unconnected-(D3-Pad1) -> GND
- D4 pad 1: unconnected-(D4-Pad1) -> GND

Commit message: less errors
Parts:
- removed D1: D_Small, Diode_SMD:D_SOD-123
- removed J3: RJ45, WS_LCSC_Connectors:RJ45_5501-88011111
- removed J4: Screw_Terminal_01x03, TerminalBlock:TerminalBlock_bornier-3_P5.08mm
- added J2: RJ45, WS_LCSC_Connectors:RJ45_5501-88011111, F.Cu at (119.4, 108.0)
- moved SW1 16.5 mm to (107.7, 89.5)
- moved C4 0.77 mm to (74.9, 81.8)
Connections:
- J1 pad A4: Net-(D1-Pad2) -> +5V
- J1 pad A9: Net-(D1-Pad2) -> +5V
- J1 pad B4: Net-(D1-Pad2) -> +5V
- J1 pad B9: Net-(D1-Pad2) -> +5V
- U3 pad 10: unconnected-(U3-Pad10) -> /PIN8_GOOD
- U3 pad 27: unconnected-(U3-Pad27) -> /PIN1_GOOD
- U3 pad 28: unconnected-(U3-Pad28) -> /PIN6_GOOD
- U3 pad 30: unconnected-(U3-Pad30) -> /PIN3_GOOD
- U3 pad 31: unconnected-(U3-Pad31) -> /PIN4_GOOD
- U3 pad 33: unconnected-(U3-Pad33) -> /PIN5_GOOD
- U3 pad 36: unconnected-(U3-Pad36) -> /PIN2_GOOD
- U3 pad 37: unconnected-(U3-Pad37) -> /PIN7_GOOD
Routing:
- net /PIN7_GOOD: track 0.00 -> 75.2 mm
- net /PIN5_GOOD: track 0.00 -> 62.5 mm
- net /PIN2_GOOD: track 0.00 -> 55.6 mm, vias 0 -> 2
- net /PIN3_GOOD: track 0.00 -> 50.5 mm
- net /PIN4_GOOD: track 0.00 -> 49.0 mm, vias 0 -> 2
- net /PIN6_GOOD: track 0.00 -> 45.0 mm, vias 0 -> 2
- net /PIN1_GOOD: track 0.00 -> 37.8 mm
- net /PIN8_GOOD: track 0.00 -> 33.8 mm, vias 0 -> 2
- net +24V: track 30.2 -> 0.00 mm
- net +5V: track 67.7 -> 38.5 mm, vias 0 -> 2
- net Net-(D1-Pad2): track 20.6 -> 0.00 mm, vias 2 -> 0
- net /SW1: track 15.2 -> 18.9 mm
- net unconnected-(U3-Pad37): track 0.95 -> 0.00 mm

Commit message: even less errors
Routing:
- net /D-: track 17.8 -> 17.1 mm
Changed lines of the file:
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@@
   (segment (start 83.82 67.31) (end 83.82 64.77) (width 0.25) (layer "F.Cu") (net 10))
   (segment (start 84.145 67.635) (end 83.82 67.31) (width 0.25) (layer "F.Cu") (net 10))
+  (segment (start 77.47 64.77) (end 81.28 64.77) (width 0.25) (layer "F.Cu") (net 11))
   (segment (start 86.425 68.905) (end 82.875 68.905) (width 0.25) (layer "F.Cu") (net 11))
   (segment (start 82.875 68.905) (end 82.55 68.58) (width 0.25) (layer "F.Cu") (net 11))
   (segment (start 76.95 65.29) (end 76.95 65.52) (width 0.25) (layer "F.Cu") (net 11))
   (segment (start 77.47 64.77) (end 76.95 65.29) (width 0.25) (layer "F.Cu") (net 11))
-  (segment (start 82.55 68.58) (end 82.55 64.77) (width 0.25) (layer "F.Cu") (net 11))
+  (segment (start 82.55 66.04) (end 82.55 68.58) (width 0.25) (layer "F.Cu") (net 11))
+  (segment (start 81.28 64.77) (end 82.55 66.04) (width 0.25) (layer "F.Cu") (net 11))
   (segment (start 75.95 66.52) (end 76.95 65.52) (width 0.25) (layer "F.Cu") (net 11))
   (segment (start 75.95 67.28) (end 75.95 66.52) (width 0.25) (layer "F.Cu") (net 11))
-  (segment (start 82.55 64.77) (end 77.47 64.77) (width 0.25) (layer "F.Cu") (net 11))
   (segment (start 76.95 65.52) (end 76.95 67.28) (width 0.25) (layer "F.Cu") (net 11))
   (segment (start 74.45 70.66) (end 74.08 71.03) (width 0.25) (layer "F.Cu") (net 13))

Commit message: labelled
Parts:
- moved D4 1.26 mm to (97.5, 78.7)
- moved R8 1.26 mm to (102.1, 78.7)
Routing:
- net Net-(R8-Pad1): track 8.68 -> 10.0 mm
Other:
- board size 100 x 100 mm -> 64.6 x 61.9 mm
- board text added: "Connected"
- board text added: "Fail"
- board text added: "Pass"
- board text added: "Run Test"
Changed lines of the file:
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@@
   )
   (footprint "Resistor_SMD:R_0402_1005Metric" (layer "F.Cu")
-    (at 102.36 77.47 180)
+    (at 102.067282 78.7 180)
     (descr "Resistor SMD 0402 (1005 Metric), square (rectangular) end terminal, IPC_7351 nominal, (Body size source: IPC-SM-782 page 72, https://www.pcb-3d.com/wordpress/wp-content/uploads/ipc-sm-782a_amendment_1_and_2.pdf), generated with kicad-footprint-generator")
     (tags "resistor")
@@
     (property "Sheetname" "")
     (attr smd)
-    (fp_text reference "R8" (at 0 -1.17) (layer "F.SilkS")
+    (fp_text reference "R8" (at 0 1.27) (layer "F.SilkS")
       (effects (font (size 1 1) (thickness 0.15)))
     )
@@
   )
   (footprint "LED_SMD:LED_0603_1608Metric" (layer "F.Cu")
-    (at 97.79 77.47)
+    (at 97.497282 78.7)
     (descr "LED SMD 0603 (1608 Metric), square (rectangular) end terminal, IPC_7351 nominal, (Body size source: http://www.tortai-tech.com/upload/download/2011102023233369053.pdf), generated with kicad-footprint-generator")
     (tags "LED")
@@
     (property "Sheetname" "")
     (attr smd)
-    (fp_text reference "D2" (at 0 -1.43) (layer "F.SilkS")
+    (fp_text reference "D2" (at 2.6275 -0.005) (layer "F.SilkS")
       (effects (font (size 1 1) (thickness 0.15)))
     )
@@
     )
   )
-  (gr_rect (start 170 60) (end 70 160) (layer "Edge.Cuts") (width 0.1) (fill none))
+  (gr_rect (start 134.62 60) (end 70 121.92) (layer "Edge.Cuts") (width 0.1) (fill none))
+  (gr_text "Run Test" (at 100.33 92.71 90) (layer "F.CrtYd")
+    (effects (font (size 1 1) (thickness 0.15)))
+  )
+  (gr_text "Fail" (at 97.79 74.93) (layer "F.CrtYd")
+    (effects (font (size 1 1) (thickness 0.15)))
+  )
+  (gr_text "Pass" (at 97.79 80.01) (layer "F.CrtYd")
+    (effects (font (size 1 1) (thickness 0.15)))
+  )
+  (gr_text "Connected" (at 101.6 102.87) (layer "F.CrtYd")
+    (effects (font (size 1 1) (thickness 0.15)))
+  )
   (segment (start 98.3 66.8) (end 98.3 66.24) (width 0.5) (layer "F.Cu") (net 1))
   (segment (start 94.305 65.095) (end 96.52 67.31) (width 0.5) (layer "F.Cu") (net 1))
@@
   (segment (start 101.695 73.505) (end 101.85 73.66) (width 0.25) (layer "F.Cu") (net 7))
   (segment (start 98.496359 73.505) (end 101.695 73.505) (width 0.25) (layer "F.Cu") (net 7))
-  (segment (start 101.85 77.47) (end 98.5775 77.47) (width 0.25) (layer "F.Cu") (net 8))
+  (segment (start 101.557282 78.7) (end 98.284782 78.7) (width 0.25) (layer "F.Cu") (net 8))
   (segment (start 77.45 67.28) (end 77.45 70.285) (width 0.25) (layer "F.Cu") (net 9))
   (segment (start 77.45 70.285) (end 78.285 71.12) (width 0.25) (layer "F.Cu") (net 9))
@@
   (segment (start 105.41 73.66) (end 108.43 70.64) (width 0.25) (layer "F.Cu") (net 18))
   (segment (start 102.87 73.66) (end 105.41 73.66) (width 0.25) (layer "F.Cu") (net 18))
-  (segment (start 108.43 71.91) (end 102.87 77.47) (width 0.25) (layer "F.Cu") (net 19))
+  (segment (start 102.577282 77.762718) (end 102.577282 78.7) (width 0.25) (layer "F.Cu") (net 19))
+  (segment (start 108.43 71.91) (end 102.577282 77.762718) (width 0.25) (layer "F.Cu") (net 19))
   (segment (start 109.25 71.91) (end 108.43 71.91) (width 0.25) (layer "F.Cu") (net 19))
   (segment (start 107.66 86.65) (end 107.66 89.46) (width 0.25) (layer "F.Cu") (net 51))

Commit message: Routing Done
Parts:
- added C6: 100nF, Capacitor_SMD:C_0402_1005Metric, F.Cu at (81.5, 82.5)
- added D1: R_LED, LED_SMD:LED_0603_1608Metric, F.Cu at (87.9, 68.3)
- added R9: 1K, Resistor_SMD:R_0402_1005Metric, F.Cu at (92.4, 63.5)
- D3: value R_LED -> LED
- SW1: footprint Button_Switch_THT:SW_PUSH_6mm -> Button_Switch_SMD:SW_SPST_TL3342
- moved U1 14.7 mm to (77.5, 76.2), turned to -90 degrees
- moved D3 14.1 mm to (87.8, 63.5)
- moved C4 12.5 mm to (87.4, 81.3)
- moved D4 11.1 mm to (87.9, 73.2)
- moved R6 11.0 mm to (92.7, 68.3)
- moved R8 10.8 mm to (92.7, 73.2)
- moved U4 9.91 mm to (93.7, 81.3)
- moved C5 8.64 mm to (100.1, 81.3)
- moved R7 3.58 mm to (101.6, 73.2)
- moved R3 3.42 mm to (97.0, 73.3)
- moved U3 3.27 mm to (114.7, 70.0)
- moved C1 2.44 mm to (101.4, 68.3)
- moved SW1 2.24 mm to (108.7, 91.4), turned to 90 degrees
- moved R5 2.22 mm to (97.0, 68.3), turned to 180 degrees
- moved R2 1.76 mm to (80.0, 69.8)
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Connections:
- D3 pad 1: GND -> +3.3V
- R6 pad 1: Net-(R6-Pad1) -> Net-(U3-Pad24)
- R6 pad 2: Net-(D3-Pad2) -> Net-(D1-Pad2)
- R8 pad 1: Net-(R8-Pad1) -> Net-(U3-Pad8)
- U1 pad 16: +3.3V -> Net-(U1-Pad16)
- U1 pad 4: +3.3V -> Net-(U1-Pad16)
- U3 pad 10: /PIN8_GOOD -> /B_SIG
- U3 pad 11: unconnected-(U3-Pad11) -> /R_SIG
- U3 pad 12: unconnected-(U3-Pad12) -> /G_SIG
- U3 pad 13: unconnected-(U3-Pad13) -> /ARGB2
- U3 pad 2: +3.3V -> Net-(U3-Pad2)
- U3 pad 23: unconnected-(U3-Pad23) -> /ARGB1
- U3 pad 24: unconnected-(U3-Pad24) -> Net-(U3-Pad24)
- U3 pad 26: unconnected-(U3-Pad26) -> /PIN8_GOOD
- U3 pad 34: unconnected-(U3-Pad34) -> /TXD
- U3 pad 35: unconnected-(U3-Pad35) -> /RXD
- U3 pad 8: Net-(R6-Pad1) -> Net-(U3-Pad8)
- U3 pad 9: Net-(R8-Pad1) -> /W_SIG
Routing:
- net /RXD: track 0.00 -> 78.2 mm, vias 0 -> 2
- net /TXD: track 0.00 -> 77.3 mm, vias 0 -> 2
- net /G_SIG: track 0.00 -> 51.7 mm
- net /R_SIG: track 0.00 -> 50.5 mm
- net /B_SIG: track 0.00 -> 50.4 mm
- net /W_SIG: track 0.00 -> 49.6 mm
- net Net-(U3-Pad24): track 0.00 -> 41.6 mm, vias 0 -> 2
- net /ARGB1: track 0.00 -> 37.8 mm
- net /ARGB2: track 0.00 -> 23.7 mm
- net Net-(R3-Pad1): track 6.85 -> 24.5 mm, vias 0 -> 2
- net /RST: track 22.3 -> 37.9 mm, vias 0 -> 4
- net +3.3V: track 71.5 -> 56.3 mm
- net Net-(U3-Pad8): track 0.00 -> 13.8 mm, vias 0 -> 2
- net Net-(U3-Pad2): track 0.00 -> 13.7 mm
- net /PIN8_GOOD: track 33.8 -> 45.4 mm
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Other:
- board size 64.6 x 61.9 mm -> 65.1 x 60.4 mm
- board text added: "ESP"
- board text added: "LED CONTROLLER TESTER MIT EAST CAMPUS RUSH 2023 W. SZETO & R. GUPTA"

Commit message: 2/20
Parts:
- moved SW1 10.2 mm to (118.9, 91.2)
- moved J2 5.32 mm to (120.3, 102.7)
- moved U2 2.05 mm to (73.4, 92.7)
- moved R4 1.52 mm to (102.3, 109.0)
- moved D2 0.78 mm to (102.1, 104.6)
Connections:
- C6 pad 2: Net-(U1-Pad16) -> GND
- D3 pad 1: +3.3V -> GND
- R9 pad 2: Net-(U3-Pad2) -> +3.3V
- U1 pad 16: Net-(U1-Pad16) -> +3.3V
- U1 pad 4: Net-(U1-Pad16) -> +3.3V
- U3 pad 16: /SW1 -> /ARGB1
- U3 pad 2: Net-(U3-Pad2) -> +3.3V
- U3 pad 23: /ARGB1 -> /SW1
Routing:
- net /TXD: track 77.3 -> 46.2 mm
- net /RXD: track 78.2 -> 48.4 mm
- net /GPI0O: track 46.1 -> 30.6 mm
- net +3.3V: track 56.3 -> 70.5 mm
- net Net-(U3-Pad2): track 13.7 -> 0.00 mm
- net /ARGB1: track 37.8 -> 26.6 mm
- net Net-(U1-Pad16): track 10.4 -> 0.00 mm
- net Net-(U3-Pad24): track 41.6 -> 32.3 mm
- net /PIN8_GOOD: track 45.4 -> 39.3 mm
- net /PIN6_GOOD: track 47.5 -> 41.9 mm
- net /PIN7_GOOD: track 77.5 -> 72.6 mm
- net /PIN1_GOOD: track 40.8 -> 35.9 mm
- net /PIN2_GOOD: track 57.8 -> 53.0 mm
- net /PIN4_GOOD: track 51.3 -> 46.4 mm
- net /PIN3_GOOD: track 53.2 -> 48.3 mm
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Other:
- board size 65.1 x 60.4 mm -> 65.1 x 54.8 mm
- board text added: "Fail T1"
- board text added: "LED CONTROLLER TESTER REV A01 MIT EAST CAMPUS RUSH 2023 W. SZETO & R. GUPTA"
- board text added: "Pass T1"
- board text added: "Pass Test 2"
- board text removed: "Connected"
- board text removed: "Fail"
- board text removed: "LED CONTROLLER TESTER MIT EAST CAMPUS RUSH 2023 W. SZETO & R. GUPTA"
- board text removed: "Pass"
