File: LED/LED.kicad_pcb (KiCad board)
At the start: 2 copper layers, 65.1 x 54.8 mm, 26 parts, among them J1 USB_C_Receptacle_USB2.0, J2 RJ45, SW1 SW_Push, U1 CH340C, U2 WeMos_D1_mini, U3 ESP32-WROOM-32D, U4 AMS1117-3.3

Commit message: small updates
Parts:
- moved R2 0.51 mm to (80.0, 69.3)
Routing:
- net +5V: track 37.0 -> 39.0 mm
Other:
- board text added: "DEVICE ON"
- board text added: "FAIL TEST 1"
- board text added: "PASS TEST 1"
- board text added: "PASS TEST 2"
- board text added: "RUN TEST"
- board text removed: "ESP"
- board text removed: "Fail T1"
- board text removed: "Pass T1"
- board text removed: "Pass Test 2"
- board text removed: "Run Test"
Changed lines of the file:
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@@
   )
   (footprint "Resistor_SMD:R_0402_1005Metric" (layer "F.Cu")
-    (at 80.01 69.85)
+    (at 80.01 69.342)
     (descr "Resistor SMD 0402 (1005 Metric), square (rectangular) end terminal, IPC_7351 nominal, (Body size source: IPC-SM-782 page 72, https://www.pcb-3d.com/wordpress/wp-content/uploads/ipc-sm-782a_amendment_1_and_2.pdf), generated with kicad-footprint-generator")
     (tags "resistor")
@@
     (property "Sheetname" "")
     (attr smd)
-    (fp_text reference "U1" (at 0 -5.9 90) (layer "F.SilkS")
+    (fp_text reference "U1" (at 0 5.842 90) (layer "F.SilkS")
       (effects (font (size 1 1) (thickness 0.15)))
     )
@@
   )
   (gr_rect (start 135.128 60) (end 70 114.808) (layer "Edge.Cuts") (width 0.1) (fill none))
-  (gr_text "ESP" (at 87.884 65.278) (layer "F.SilkS")
+  (gr_text "DEVICE ON" (at 87.884 65.278) (layer "F.SilkS")
     (effects (font (size 1 1) (thickness 0.2)))
   )
-  (gr_text "Fail T1" (at 87.63 70.104) (layer "F.SilkS")
+  (gr_text "RUN TEST" (at 122.872 91.186 270) (layer "F.SilkS")
+    (effects (font (size 1 1) (thickness 0.15)))
+  )
+  (gr_text "FAIL TEST 1" (at 87.63 70.104) (layer "F.SilkS")
     (effects (font (size 1 1) (thickness 0.2)))
   )
@@
     (effects (font (size 1 1) (thickness 0.2)))
   )
-  (gr_text "Pass T1" (at 87.63 74.676) (layer "F.SilkS")
+  (gr_text "PASS TEST 1" (at 87.63 74.676) (layer "F.SilkS")
     (effects (font (size 1 1) (thickness 0.2)))
   )
-  (gr_text "Run Test" (at 122.872 91.186 270) (layer "F.CrtYd")
-    (effects (font (size 1 1) (thickness 0.15)))
-  )
-  (gr_text "Pass Test 2" (at 102.1955 103.373) (layer "F.CrtYd")
+  (gr_text "PASS TEST 2" (at 102.1955 103.373) (layer "F.SilkS")
     (effects (font (size 1 1) (thickness 0.15)))
   )
@@
   (segment (start 98.806 73.152) (end 98.552 73.406) (width 0.25) (layer "B.Cu") (net 3))
   (segment (start 98.552 73.406) (end 98.552 78.994) (width 0.25) (layer "B.Cu") (net 3))
-  (segment (start 86.601 81.28) (end 86.601 82.537) (width 0.25) (layer "F.Cu") (net 4))
   (segment (start 89.14 83.58) (end 88.392 84.328) (width 0.25) (layer "F.Cu") (net 4))
+  (segment (start 78.6 68.11) (end 79.07 68.58) (width 0.25) (layer "F.Cu") (net 4))
   (segment (start 90.576 83.58) (end 89.14 83.58) (width 0.25) (layer "F.Cu") (net 4))
-  (segment (start 83.058 69.088) (end 84.328 70.358) (width 0.25) (layer "F.Cu") (net 4))
   (segment (start 74.444596 63.797598) (end 74.444596 66.04) (width 0.25) (layer "F.Cu") (net 4))
+  (segment (start 85.3375 80.0165) (end 85.344 80.023) (width 0.25) (layer "F.Cu") (net 4))
+  (segment (start 74.444596 66.04) (end 73.8 66.684596) (width 0.25) (layer "F.Cu") (net 4))
+  (segment (start 85.344 80.023) (end 85.344 82.042) (width 0.25) (layer "F.Cu") (net 4))
+  (segment (start 73.8 66.684596) (end 73.8 67.28) (width 0.25) (layer "F.Cu") (net 4))
+  (segment (start 78.6 67.28) (end 78.6 68.11) (width 0.25) (layer "F.Cu") (net 4))
+  (segment (start 82.55 68.58) (end 84.328 70.358) (width 0.25) (layer "F.Cu") (net 4))
+  (segment (start 78.6 66.684596) (end 78.6 67.28) (width 0.25) (layer "F.Cu") (net 4))
   (segment (start 84.328 70.358) (end 84.328 79.007) (width 0.25) (layer "F.Cu") (net 4))
-  (segment (start 74.444596 66.04) (end 73.8 66.684596) (width 0.25) (layer "F.Cu") (net 4))
-  (segment (start 78.6 68.11) (end 79.578 69.088) (width 0.25) (layer "F.Cu") (net 4))
-  (segment (start 79.578 69.088) (end 83.058 69.088) (width 0.25) (layer "F.Cu") (net 4))
-  (segment (start 73.8 66.684596) (end 73.8 67.28) (width 0.25) (layer "F.Cu") (net 4))
-  (segment (start 86.601 82.537) (end 86.614 82.55) (width 0.25) (layer "F.Cu") (net 4))
-  (segment (start 84.328 79.007) (end 86.601 81.28) (width 0.25) (layer "F.Cu") (net 4))
-  (segment (start 78.6 66.684596) (end 78.6 67.28) (width 0.25) (layer "F.Cu") (net 4))
-  (segment (start 78.6 67.28) (end 78.6 68.11) (width 0.25) (layer "F.Cu") (net 4))
   (segment (start 77.47 63.5) (end 77.47 65.554596) (width 0.25) (layer "F.Cu") (net 4))
-  (segment (start 86.614 82.55) (end 86.614 82.4605) (width 0.25) (layer "F.Cu") (net 4))
+  (segment (start 85.3375 80.0165) (end 86.601 81.28) (width 0.25) (layer "F.Cu") (net 4))
   (segment (start 74.742194 63.5) (end 74.444596 63.797598) (width 0.25) (layer "F.Cu") (net 4))
   (segment (start 77.47 65.554596) (end 78.6 66.684596) (width 0.25) (layer "F.Cu") (net 4))
+  (segment (start 79.07 68.58) (end 82.55 68.58) (width 0.25) (layer "F.Cu") (net 4))
+  (segment (start 84.328 79.007) (end 85.3375 80.0165) (width 0.25) (layer "F.Cu") (net 4))
   (via (at 74.742194 63.5) (size 0.8) (drill 0.4) (layers "F.Cu" "B.Cu") (net 4))
+  (via (at 85.344 82.042) (size 0.8) (drill 0.4) (layers "F.Cu" "B.Cu") (net 4))
   (via (at 88.392 84.328) (size 0.8) (drill 0.4) (layers "F.Cu" "B.Cu") (net 4))
   (via (at 77.47 63.5) (size 0.8) (drill 0.4) (layers "F.Cu" "B.Cu") (net 4))
-  (via (at 86.614 82.4605) (size 0.8) (drill 0.4) (layers "F.Cu" "B.Cu") (net 4))
-  (segment (start 86.614 82.55) (end 88.392 84.328) (width 0.25) (layer "B.Cu") (net 4))
+  (segment (start 86.106 82.042) (end 88.392 84.328) (width 0.25) (layer "B.Cu") (net 4))
+  (segment (start 85.344 82.042) (end 86.106 82.042) (width 0.25) (layer "B.Cu") (net 4))
   (segment (start 74.742194 63.5) (end 77.47 63.5) (width 0.25) (layer "B.Cu") (net 4))
-  (segment (start 86.614 82.4605) (end 86.614 82.55) (width 0.25) (layer "B.Cu") (net 4))
   (segment (start 98.0185 107.95) (end 96.233 107.95) (width 0.25) (layer "F.Cu") (net 5))
   (segment (start 101.3205 104.648) (end 98.0185 107.95) (width 0.25) (layer "F.Cu") (net 5))
@@
   (segment (start 92.0995 73.152) (end 92.1875 73.24) (width 0.25) (layer "F.Cu") (net 7))
   (segment (start 88.659 73.152) (end 92.0995 73.152) (width 0.25) (layer "F.Cu") (net 7))
-  (segment (start 79.5 69.85) (end 79.248 69.85) (width 0.25) (layer "F.Cu") (net 8))
-  (segment (start 79.248 69.85) (end 77.45 68.052) (width 0.25) (layer "F.Cu") (net 8))
+  (segment (start 78.74 69.342) (end 79.5 69.342) (width 0.25) (layer "F.Cu") (net 8))
   (segment (start 77.45 68.052) (end 77.45 67.28) (width 0.25) (layer "F.Cu") (net 8))
+  (segment (start 77.45 68.052) (end 78.74 69.342) (width 0.25) (layer "F.Cu") (net 8))
   (segment (start 76.835 73.725) (end 76.6612 73.5512) (width 0.77) (layer "F.Cu") (net 9))
   (segment (start 76.6612 73.5512) (end 76.6612 68.626763) (width 0.77) (layer "F.Cu") (net 9))

Commit message: Final PCB Version 1
Parts:
- added G***: LOGO, Castle:Castle2, B.Cu at (103.1, 87.1)
