File: LED/LED.kicad_sch (KiCad schematic)
At the start: 25 parts, among them J1 USB_C_Receptacle_USB2.0, J2 RJ45, J3 RJ45, J4 Screw_Terminal_01x03, U1 CH340C, U2 WeMos_D1_mini, U3 ESP32-WROOM-32D, U4 AMS1117-3.3

Commit message: 2 ethernet
Parts:
- added SW1: SW_Push, Button_Switch_THT:SW_PUSH_6mm, symbol Switch:SW_Push
Connections:
- net GND: now also SW1.2
- net SW1: now reaches U3.16 (IO13)
- net SW1: now also SW1.1
Other:
- note added: "Button to Start Test"
- note added: "Ethernet Pin Tester"
- note added: "Ethernet for Power"
- note added: "MCU Connector"
- note added: "Microcontroller"
- note added: "Power - USB C"
- note added: "Screw Terminal Power Input"
- note added: "USB Serial Converter"
- moved on the sheet: C1, C2, C3, C4, C5, D2, D3, D4, J2, J3, J4, R4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

Commit message: 2/12
first draft
Parts:
- removed J2: RJ45, WS_LCSC_Connectors:RJ45_5501-88011111, symbol Connector:RJ45
Connections:
- net PIN1_GOOD: no longer names the net of U3.10 (IO25)
- net PIN2_GOOD: no longer names the net of U3.37 (IO23)
- net PIN3_GOOD: no longer names the net of U3.36 (IO22)
- net PIN4_GOOD: no longer names the net of U3.33 (IO21)
- net PIN5_GOOD: no longer names the net of U3.31 (IO19)
- net PIN6_GOOD: no longer names the net of U3.30 (IO18)
- net PIN7_GOOD: no longer names the net of U3.28 (IO17)
- net PIN8_GOOD: no longer names the net of U3.27 (IO16)
Other:
- note added: "Voltage Regulator"
- note removed: "Ethernet Pin Tester"
- moved on the sheet: D2, J3, R4, U2

Commit message: to gnd
Connections:
- net GND: now also D3.1 (K), D4.1 (K)
Other:
- moved on the sheet: R8
Changed lines of the file:
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@@
+    (stroke (width 0) (type default) (color 0 0 0 0))
+  )
+  (wire (pts (xy 213.36 95.25) (xy 214.63 95.25))
     (stroke (width 0) (type default) (color 0 0 0 0))
   )
@@
     (stroke (width 0) (type default) (color 0 0 0 0))
   )
-  (wire (pts (xy 210.82 95.25) (xy 214.63 95.25))
-    (stroke (width 0) (type default) (color 0 0 0 0))
-  )
   (wire (pts (xy 39.37 116.84) (xy 39.37 119.38))
     (stroke (width 0) (type default) (color 0 0 0 0))
@@
     (stroke (width 0) (type default) (color 0 0 0 0))
   )
-  (wire (pts (xy 185.42 95.25) (xy 205.74 95.25))
+  (wire (pts (xy 185.42 95.25) (xy 208.28 95.25))
     (stroke (width 0) (type default) (color 0 0 0 0))
   )
@@
     (stroke (width 0) (type default) (color 0 0 0 0))
   )
+  (wire (pts (xy 222.25 95.25) (xy 222.25 99.06))
+    (stroke (width 0) (type default) (color 0 0 0 0))
+  )
   (wire (pts (xy 39.37 106.68) (xy 39.37 109.22))
     (stroke (width 0) (type default) (color 0 0 0 0))
@@
   )
   (polyline (pts (xy 128.27 115.57) (xy 128.27 13.97))
+    (stroke (width 0) (type default) (color 0 0 0 0))
+  )
+  (wire (pts (xy 207.01 92.71) (xy 204.47 92.71))
+    (stroke (width 0) (type default) (color 0 0 0 0))
+  )
+  (wire (pts (xy 207.01 81.28) (xy 207.01 92.71))
     (stroke (width 0) (type default) (color 0 0 0 0))
   )
@@
     (pin "2")
   )
+  (symbol (lib_id "power:GND") (at 222.25 99.06 0) (unit 1)
+    (in_bom yes) (on_board yes) (fields_autoplaced)
+    (property "Reference" "#PWR?" (id 0) (at 222.25 105.41 0)
+      (effects (font (size 1.27 1.27)) hide)
+    )
+    (property "Value" "GND" (id 1) (at 222.25 104.14 0))
+    (property "Footprint" "" (id 2) (at 222.25 99.06 0)
+      (effects (font (size 1.27 1.27)) hide)
+    )
+    (property "Datasheet" "" (id 3) (at 222.25 99.06 0)
+      (effects (font (size 1.27 1.27)) hide)
+    )
+    (pin "1")
+  )
   (symbol (lib_id "Device:R_Small") (at 195.58 39.37 0) (unit 1)
     (in_bom yes) (on_board yes) (fields_autoplaced)
@@
     (pin "1")
   )
-  (symbol (lib_id "Device:R_Small") (at 208.28 95.25 90) (unit 1)
+  (symbol (lib_id "Device:R_Small") (at 210.82 95.25 90) (unit 1)
     (in_bom yes) (on_board yes)
-    (property "Reference" "R8" (id 0) (at 208.28 90.17 90))
-    (property "Value" "330" (id 1) (at 208.28 92.71 90))
-    (property "Footprint" "Resistor_SMD:R_0402_1005Metric" (id 2) (at 208.28 95.25 0)
-      (effects (font (size 1.27 1.27)) hide)
-    )
-    (property "Datasheet" "~" (id 3) (at 208.28 95.25 0)
+    (property "Reference" "R8" (id 0) (at 210.82 90.17 90))
+    (property "Value" "330" (id 1) (at 210.82 92.71 90))
+    (property "Footprint" "Resistor_SMD:R_0402_1005Metric" (id 2) (at 210.82 95.25 0)
+      (effects (font (size 1.27 1.27)) hide)
+    )
+    (property "Datasheet" "~" (id 3) (at 210.82 95.25 0)
       (effects (font (size 1.27 1.27)) hide)
     )
@@
     (pin "2")
   )
+  (symbol (lib_id "power:GND") (at 207.01 81.28 180) (unit 1)
+    (in_bom yes) (on_board yes) (fields_autoplaced)
+    (property "Reference" "#PWR?" (id 0) (at 207.01 74.93 0)
+      (effects (font (size 1.27 1.27)) hide)
+    )
+    (property "Value" "GND" (id 1) (at 207.01 76.2 0))
+    (property "Footprint" "" (id 2) (at 207.01 81.28 0)
+      (effects (font (size 1.27 1.27)) hide)
+    )
+    (property "Datasheet" "" (id 3) (at 207.01 81.28 0)
+      (effects (font (size 1.27 1.27)) hide)
+    )
+    (pin "1")
+  )
   (symbol (lib_id "Regulator_Linear:AMS1117-3.3") (at 255.27 93.98 0) (unit 1)
     (in_bom yes) (on_board yes) (fields_autoplaced)
@@
       (reference "#PWR0123") (unit 1) (value "GND") (footprint "")
     )
+    (path "/5d188542-8245-4317-8d12-db43ed8ffd1c"
+      (reference "#PWR?") (unit 1) (value "GND") (footprint "")
+    )
+    (path "/d56db942-7cf8-4b42-8a8d-1c71c8215aaa"
+      (reference "#PWR?") (unit 1) (value "GND") (footprint "")
+    )
     (path "/cac6a1ff-2c1b-4280-80a9-10e16e37f5dc"

Commit message: less errors
Parts:
- removed D1: D_Small, Diode_SMD:D_SOD-123, symbol Device:D_Small
- removed J3: RJ45, WS_LCSC_Connectors:RJ45_5501-88011111, symbol Connector:RJ45
- removed J4: Screw_Terminal_01x03, TerminalBlock:TerminalBlock_bornier-3_P5.08mm, symbol Connector:Screw_Terminal_01x03
- added J2: RJ45, WS_LCSC_Connectors:RJ45_5501-88011111, symbol Connector:RJ45
Connections:
- net +5V: now also J1.A4 (VBUS), J1.A9 (VBUS), J1.B4 (VBUS), J1.B9 (VBUS)
- net PIN8_GOOD: now reaches U3.10 (IO25)
- net PIN8_GOOD: now also J2.8
- net PIN1_GOOD: now reaches U3.27 (IO16)
- net PIN1_GOOD: now also J2.1
- net PIN6_GOOD: now reaches U3.28 (IO17)
- net PIN6_GOOD: now also J2.6
- net PIN3_GOOD: now reaches U3.30 (IO18)
- net PIN3_GOOD: now also J2.3
- net PIN4_GOOD: now reaches U3.31 (IO19)
- net PIN4_GOOD: now also J2.4
- net PIN5_GOOD: now reaches U3.33 (IO21)
- net PIN5_GOOD: now also J2.5
- net PIN2_GOOD: now reaches U3.36 (IO22)
- net PIN2_GOOD: now also J2.2
- net PIN7_GOOD: now reaches U3.37 (IO23)
- net PIN7_GOOD: now also J2.7
Other:
- note added: "Ethernet Pin Tester"
- note removed: "Ethernet for Power"
- note removed: "Screw Terminal Power Input"
- moved on the sheet: C4, C5, U4

Commit message: Routing Done
Parts:
- added C6: 100nF, Capacitor_SMD:C_0402_1005Metric, symbol Device:C_Small
- added D1: R_LED, LED_SMD:LED_0603_1608Metric, symbol Device:LED
- added R9: 1K, Resistor_SMD:R_0402_1005Metric, symbol Device:R_Small
- D3: value R_LED -> LED
- SW1: footprint Button_Switch_THT:SW_PUSH_6mm -> Button_Switch_SMD:SW_SPST_TL3342; LCSC (none) -> C318884
Connections:
- net +3.3V: now also D3.1 (K), C6.1; no longer U1.16 (VCC), U1.4 (V3), U3.2 (VDD)
- net ARGB1: now also U3.23 (IO15)
- net ARGB2: now also U3.13 (IO14)
- net B_SIG: now also U3.10 (IO25)
- net GND: now also D1.1 (K); no longer D3.1 (K)
- net G_SIG: now also U3.12 (IO27)
- net PIN8_GOOD: now also U3.26 (IO4); no longer U3.10 (IO25)
- net RXD: now also U3.35 (TXD0/IO1)
- net R_SIG: now also U3.11 (IO26)
- net TXD: now also U3.34 (RXD0/IO3)
- net W_SIG: now also U3.9 (IO33)
- net at U3.24 (IO2): now also R6.1
- net at U3.8 (IO32): now also R8.1; no longer R6.1
- net at D3.2 (A): now also R9.1; no longer R6.2
- new net: C6.2, U1.16 (VCC), U1.4 (V3)
- new net: R9.2, U3.2 (VDD)
- new net: D1.2 (A), R6.2
- no-connect marks 0 -> 26
Other:
- moved on the sheet: D4, R8

Commit message: 2/20
Connections:
- net +3.3V: now also R9.2, U1.16 (VCC), U1.4 (V3), U3.2 (VDD); no longer D3.1 (K)
- net ARGB1: now also U3.16 (IO13); no longer U3.23 (IO15)
- net GND: now also C6.2, D3.1 (K)
- net SW1: now also U3.23 (IO15); no longer U3.16 (IO13)
Other:
- moved on the sheet: C6, D3, R9

Commit message: Final PCB Version 1
Parts:
- C1, C3, C6: LCSC (none) -> C1525
- C2, C4, C5: LCSC (none) -> C19702
- D1: LCSC (none) -> C2286
- D2, D3, D4: LCSC (none) -> C72043
- R1, R2: LCSC (none) -> C25905
- R3: LCSC (none) -> C25091
- R4, R9: LCSC (none) -> C11702
- R5, R7: LCSC (none) -> C25744
- R6, R8: LCSC (none) -> C25104
- U4: LCSC (none) -> C6186
Changed lines of the file:
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@@
+      (effects (font (size 1.27 1.27)) hide)
+    )
+    (property "LCSC" "C25905" (id 4) (at 57.15 36.83 0)
       (effects (font (size 1.27 1.27)) hide)
     )
@@
       (effects (font (size 1.27 1.27)) hide)
     )
+    (property "LCSC" "C19702" (id 4) (at 241.3 64.77 0)
+      (effects (font (size 1.27 1.27)) hide)
+    )
     (pin "1")
     (pin "2")
@@
   (symbol (lib_id "power:GND") (at 180.34 30.48 0) (unit 1)
     (in_bom yes) (on_board yes)
-    (property "Reference" "#PWR?" (id 0) (at 180.34 36.83 0)
+    (property "Reference" "#PWR0115" (id 0) (at 180.34 36.83 0)
       (effects (font (size 1.27 1.27)) hide)
     )
@@
       (effects (font (size 1.27 1.27)) hide)
     )
+    (property "LCSC" "C1525" (id 4) (at 158.75 26.67 0)
+      (effects (font (size 1.27 1.27)) hide)
+    )
     (pin "1")
     (pin "2")
@@
     )
     (property "Datasheet" "~" (id 3) (at 180.34 26.67 0)
+      (effects (font (size 1.27 1.27)) hide)
+    )
+    (property "LCSC" "C72043" (id 4) (at 180.34 26.67 0)
       (effects (font (size 1.27 1.27)) hide)
     )
@@
       (effects (font (size 1.27 1.27)) hide)
     )
+    (property "LCSC" "C25744" (id 4) (at 195.58 39.37 0)
+      (effects (font (size 1.27 1.27)) hide)
+    )
     (pin "1")
     (pin "2")
@@
       (effects (font (size 1.27 1.27)) hide)
     )
+    (property "LCSC" "C25104" (id 4) (at 204.47 46.99 0)
+      (effects (font (size 1.27 1.27)) hide)
+    )
     (pin "1")
     (pin "2")
@@
     )
     (property "Datasheet" "~" (id 3) (at 101.6 27.94 0)
+      (effects (font (size 1.27 1.27)) hide)
+    )
+    (property "LCSC" "C1525" (id 4) (at 101.6 27.94 0)
       (effects (font (size 1.27 1.27)) hide)
     )
@@
       (effects (font (size 1.27 1.27)) hide)
     )
+    (property "LCSC" "C25104" (id 4) (at 204.47 92.71 0)
+      (effects (font (size 1.27 1.27)) hide)
+    )
     (pin "1")
     (pin "2")
@@
       (effects (font (size 1.27 1.27)) hide)
     )
+    (property "LCSC" "C11702" (id 4) (at 180.34 20.32 0)
+      (effects (font (size 1.27 1.27)) hide)
+    )
     (pin "1")
     (pin "2")
@@
     )
     (property "Datasheet" "~" (id 3) (at 269.24 64.77 0)
+      (effects (font (size 1.27 1.27)) hide)
+    )
+    (property "LCSC" "C19702" (id 4) (at 269.24 64.77 0)
       (effects (font (size 1.27 1.27)) hide)
     )
@@
       (effects (font (size 1.27 1.27)) hide)
     )
+    (property "LCSC" "C25091" (id 4) (at 113.03 55.88 0)
+      (effects (font (size 1.27 1.27)) hide)
+    )
     (pin "1")
     (pin "2")
@@
       (effects (font (size 1.27 1.27)) hide)
     )
+    (property "LCSC" "C19702" (id 4) (at 146.05 26.67 0)
+      (effects (font (size 1.27 1.27)) hide)
+    )
     (pin "1")
     (pin "2")
@@
   (symbol (lib_id "power:GND") (at 101.6 30.48 0) (unit 1)
     (in_bom yes) (on_board yes)
-    (property "Reference" "#PWR?" (id 0) (at 101.6 36.83 0)
+    (property "Reference" "#PWR0113" (id 0) (at 101.6 36.83 0)
       (effects (font (size 1.27 1.27)) hide)
     )
@@
     )
     (property "Datasheet" "~" (id 3) (at 52.07 39.37 0)
+      (effects (font (size 1.27 1.27)) hide)
+    )
+    (property "LCSC" "C25905" (id 4) (at 52.07 39.37 0)
       (effects (font (size 1.27 1.27)) hide)
     )
@@
       (effects (font (size 1.27 1.27)) hide)
     )
+    (property "LCSC" "C11702" (id 4) (at 93.98 115.57 0)
+      (effects (font (size 1.27 1.27)) hide)
+    )
     (pin "1")
     (pin "2")
@@
     )
     (property "Datasheet" "~" (id 3) (at 135.89 46.99 0)
+      (effects (font (size 1.27 1.27)) hide)
+    )
+    (property "LCSC" "C1525" (id 4) (at 135.89 46.99 0)
       (effects (font (size 1.27 1.27)) hide)
     )
@@
       (effects (font (size 1.27 1.27)) hide)
     )
+    (property "LCSC" "C2286" (id 4) (at 214.63 46.99 0)
+      (effects (font (size 1.27 1.27)) hide)
+    )
     (pin "1")
     (pin "2")
@@
     )
     (property "Datasheet" "~" (id 3) (at 135.89 35.56 0)
+      (effects (font (size 1.27 1.27)) hide)
+    )
+    (property "LCSC" "C25744" (id 4) (at 135.89 35.56 0)
       (effects (font (size 1.27 1.27)) hide)
     )
@@
       (effects (font (size 1.27 1.27)) hide)
     )
+    (property "LCSC" "C6186" (id 4) (at 255.27 59.69 0)
+      (effects (font (size 1.27 1.27)) hide)
+    )
     (pin "1")
     (pin "2")
@@
       (effects (font (size 1.27 1.27)) hide)
     )
+    (property "LCSC" "C72043" (id 4) (at 212.09 92.71 0)
+      (effects (font (size 1.27 1.27)) hide)
+    )
     (pin "1")
     (pin "2")
@@
     )
     (property "Datasheet" "~" (id 3) (at 93.98 106.68 0)
+      (effects (font (size 1.27 1.27)) hide)
+    )
+    (property "LCSC" "C72043" (id 4) (at 93.98 106.68 0)
       (effects (font (size 1.27 1.27)) hide)
     )
@@
       (reference "#PWR0112") (unit 1) (value "GND") (footprint "")
     )
+    (path "/af745b82-8ae4-4876-9550-1f5cace244cd"
+      (reference "#PWR0113") (unit 1) (value "GND") (footprint "")
+    )
     (path "/6cc357c4-5360-4650-bd3e-0fab01e95631"
       (reference "#PWR0114") (unit 1) (value "GND") (footprint "")
     )
+    (path "/34e68c8d-9571-47f5-89bf-df9a83fdaf52"
+      (reference "#PWR0115") (unit 1) (value "GND") (footprint "")
+    )
     (path "/d08081dc-8051-4c25-b64d-1b7c7810e4eb"
       (reference "#PWR0118") (unit 1) (value "GND") (footprint "")
@@
       (reference "#PWR0125") (unit 1) (value "GND") (footprint "")
     )
-    (path "/34e68c8d-9571-47f5-89bf-df9a83fdaf52"
-      (reference "#PWR?") (unit 1) (value "GND") (footprint "")
-    )
-    (path "/af745b82-8ae4-4876-9550-1f5cace244cd"
-      (reference "#PWR?") (unit 1) (value "GND") (footprint "")
-    )
     (path "/cac6a1ff-2c1b-4280-80a9-10e16e37f5dc"
